File: HW15/hw15/hw15.kicad_pcb (KiCad board)
At the start: 2 copper layers, 1 part

Commit message: done with pcb
Parts:
- removed REF**: TSOT-23-6_HandSoldering, Package_TO_SOT_SMD:TSOT-23-6_HandSoldering
- added C1: 22uF, Capacitor_SMD:CP_Elec_8x6.2, F.Cu at (168.6, 55.0)
- added C2: 22uF, Capacitor_SMD:CP_Elec_8x6.2, F.Cu at (195.0, 67.0)
- added D1: D_Schottky, Diode_SMD:D_3220_8050Metric_Pad2.65x5.15mm_HandSolder, F.Cu at (179.7, 55.0)
- added D2: red, LED_THT:LED_D2.0mm_W4.8mm_H2.5mm_FlatTop, F.Cu at (156.5, 69.0)
- added J1: Conn_01x03_Pin, Connector_PinSocket_2.54mm:PinSocket_1x03_P2.54mm_Vertical, F.Cu at (160.0, 53.5)
- added L1: 4.7uH, Inductor_SMD:L_1206_3216Metric, F.Cu at (188.4, 55.0)
- added R1: 110k, Resistor_SMD:R_0805_2012Metric_Pad1.20x1.40mm_HandSolder, F.Cu at (180.5, 67.5)
- added R2: 15k, Resistor_SMD:R_0805_2012Metric_Pad1.20x1.40mm_HandSolder, F.Cu at (180.5, 63.0)
- added R3: 20k, Resistor_SMD:R_0805_2012Metric_Pad1.20x1.40mm_HandSolder, F.Cu at (194.5, 58.5)
- added R4: 1k, Resistor_SMD:R_0805_2012Metric_Pad1.20x1.40mm_HandSolder, F.Cu at (156.5, 62.5)
- added U1: MT3608, Package_TO_SOT_SMD:SOT-23-6, F.Cu at (188.4, 60.5)
Routing:
- net VCC: track 0.00 -> 61.1 mm
- net +5V: track 0.00 -> 45.8 mm
- net Net-(U1-FB): track 0.00 -> 10.9 mm
- net Net-(D1A-A): track 0.00 -> 9.60 mm
- net Net-(D2-K): track 0.00 -> 8.49 mm
- net Net-(U1-OC): track 0.00 -> 5.00 mm
- added copper zone on F.Cu, net GND
Other:
- board outline added: 46 x 23 mm
