File: HW15/hw15/hw15.kicad_sch (KiCad schematic)
At the start: 0 parts

Commit message: 11
Parts:
- added C1, C2: 22uF, symbol Device:C
- added D1: D_Schottky, symbol Device:D_Schottky_Dual_CommonAnode_AKK_Split
- added D2: red, symbol Device:LED
- added J1: Conn_01x03_Pin, symbol Connector:Conn_01x03_Pin
- added L1: 4.7uH, symbol Device:L_Small
- added R1: 110k, symbol Device:R_US
- added R2: 15k, symbol Device:R_US
- added R3: 20k, symbol Device:R_US
- added R4: 1k, symbol Device:R_US
- added U1: MT3608, Package_TO_SOT_SMD:SOT-23-6, symbol Regulator_Switching:MT3608
Connections:
- new net: R3.1, U1.6 (OC)
- new net: D2.1 (K), R4.1
- new net: D1.1 (A), L1.2, U1.1 (SW)
- new net: R1.2, R2.1, U1.3 (FB)
- new net +5V: C1.1, D1.2 (K), D2.2 (A), J1.3 (Pin_3), R1.1
- new net GND: C1.2, C2.2, J1.2 (Pin_2), R2.2, R3.2, R4.2, U1.2 (GND)
- new net VCC: C2.1, J1.1 (Pin_1), L1.1, U1.4 (EN), U1.5 (VIN)

Commit message: done with pcb
Parts:
- C1, C2: footprint (none) -> Capacitor_SMD:CP_Elec_8x6.2
- D1: footprint (none) -> Diode_SMD:D_3220_8050Metric_Pad2.65x5.15mm_HandSolder
- D2: footprint (none) -> LED_THT:LED_D2.0mm_W4.8mm_H2.5mm_FlatTop
- J1: footprint (none) -> Connector_PinSocket_2.54mm:PinSocket_1x03_P2.54mm_Vertical
- L1: footprint (none) -> Inductor_SMD:L_1206_3216Metric
- R1, R2, R3, R4: footprint (none) -> Resistor_SMD:R_0805_2012Metric_Pad1.20x1.40mm_HandSolder
Changed lines of the file:
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@@
 			)
 		)
-		(property "Footprint" ""
+		(property "Footprint" "Resistor_SMD:R_0805_2012Metric_Pad1.20x1.40mm_HandSolder"
 			(at 171.196 89.154 90)
 			(effects
@@
 			)
 		)
-		(property "Footprint" ""
+		(property "Footprint" "LED_THT:LED_D2.0mm_W4.8mm_H2.5mm_FlatTop"
 			(at 182.88 91.44 0)
 			(effects
@@
 			)
 		)
-		(property "Footprint" ""
+		(property "Footprint" "Capacitor_SMD:CP_Elec_8x6.2"
 			(at 107.6452 95.25 0)
 			(effects
@@
 			)
 		)
-		(property "Footprint" ""
+		(property "Footprint" "Inductor_SMD:L_1206_3216Metric"
 			(at 139.7 76.2 0)
 			(effects
@@
 			)
 		)
-		(property "Footprint" ""
+		(property "Footprint" "Connector_PinSocket_2.54mm:PinSocket_1x03_P2.54mm_Vertical"
 			(at 78.74 91.44 0)
 			(effects
@@
 			)
 		)
-		(property "Footprint" ""
+		(property "Footprint" "Diode_SMD:D_3220_8050Metric_Pad2.65x5.15mm_HandSolder"
 			(at 147.32 78.74 0)
 			(effects
@@
 			)
 		)
-		(property "Footprint" ""
+		(property "Footprint" "Resistor_SMD:R_0805_2012Metric_Pad1.20x1.40mm_HandSolder"
 			(at 145.796 118.364 90)
 			(effects
@@
 			)
 		)
-		(property "Footprint" ""
+		(property "Footprint" "Resistor_SMD:R_0805_2012Metric_Pad1.20x1.40mm_HandSolder"
 			(at 183.896 101.854 90)
 			(effects
@@
 			)
 		)
-		(property "Footprint" ""
+		(property "Footprint" "Capacitor_SMD:CP_Elec_8x6.2"
 			(at 120.3452 95.25 0)
 			(effects
@@
 			)
 		)
-		(property "Footprint" ""
+		(property "Footprint" "Resistor_SMD:R_0805_2012Metric_Pad1.20x1.40mm_HandSolder"
 			(at 145.796 108.204 90)
 			(effects
